Commit message: effort and diff drive stable

File: src/apriltag_slam/urdf/robot.urdf.xacro (robot description, xacro)
@@ -12,13 +12,10 @@
   <xacro:property name="wheel_width"  value="0.05"/>
   <xacro:property name="wheel_mass"   value="3.1"/>
-  <xacro:property name="wheelbase" value="0.6"/>
-  <xacro:property name="track"     value="0.6"/>
-  <xacro:property name="cam_size" value="0.125"/>
+  <xacro:property name="track" value="0.6"/>
+  <xacro:property name="cam_size" value="0.05"/>
   <xacro:macro name="box_inertia" params="m x y z">
     <inertial>
       <mass value="${m}"/>
-      <inertia ixx="${m*(y*y+z*z)/12}" ixy="0" ixz="0"
-               iyy="${m*(x*x+z*z)/12}" iyz="0"
-               izz="${m*(x*x+y*y)/12}"/>
+      <inertia ixx="${m*(y*y+z*z)/12}" iyy="${m*(x*x+z*z)/12}" izz="${m*(x*x+y*y)/12}" ixy="0" ixz="0" iyz="0"/>
     </inertial>
   </xacro:macro>
@@ -26,78 +23,69 @@
     <inertial>
       <mass value="${m}"/>
-      <inertia ixx="${m*(3*r*r+h*h)/12}" ixy="0" ixz="0"
-               iyy="${m*(3*r*r+h*h)/12}" iyz="0"
-               izz="${m*r*r/2}"/>
+      <inertia ixx="${m*(3*r*r+h*h)/12}" iyy="${m*(3*r*r+h*h)/12}" izz="${m*r*r/2}" ixy="0" ixz="0" iyz="0"/>
     </inertial>
   </xacro:macro>
-  <link name="base_footprint"/>
-  <joint name="base_joint" type="fixed">
-    <parent link="base_footprint"/>
-    <child link="base_link"/>
-    <origin xyz="0 0 ${wheel_radius + base_height/2}" rpy="0 0 0"/>
-  </joint>
   <link name="base_link">
     <xacro:box_inertia m="${base_mass}" x="${base_length}" y="${base_width}" z="${base_height}"/>
     <visual>
+      <origin xyz="0 0 ${base_height/2 + wheel_radius}" rpy="0 0 0"/>
       <geometry><box size="${base_length} ${base_width} ${base_height}"/></geometry>
       <material name="blue"/>
     </visual>
     <collision>
+      <origin xyz="0 0 ${base_height/2 + wheel_radius}" rpy="0 0 0"/>
       <geometry><box size="${base_length} ${base_width} ${base_height}"/></geometry>
     </collision>
   </link>
-  <xacro:macro name="rear_wheel" params="prefix y_offset">
-    <link name="${prefix}_wheel_link">
+  <link name="front_caster">
+    <visual>
+      <geometry><sphere radius="${wheel_radius}"/></geometry>
+      <material name="black"/>
+    </visual>
+    <collision>
+      <geometry><sphere radius="${wheel_radius}"/></geometry>
+    </collision>
+    <inertial>
+      <mass value="0.1"/>
+      <inertia ixx="0.0001" ixy="0.0" ixz="0.0" iyy="0.0001" iyz="0.0" izz="0.0001"/>
+    </inertial>
+  </link>
+  <joint name="caster_joint" type="fixed">
+    <parent link="base_link"/>
+    <child link="front_caster"/>
+    <origin xyz="${base_length/3} 0 ${wheel_radius}"/>
+  </joint>
+  <gazebo reference="front_caster">
+    <mu1 value="0.001"/>
+    <mu2 value="0.001"/>
+  </gazebo>
+  <xacro:macro name="wheel" params="name y">
+    <link name="${name}_wheel_link">
       <xacro:cylinder_inertia m="${wheel_mass}" r="${wheel_radius}" h="${wheel_width}"/>
       <visual>
+        <origin xyz="0 0 0" rpy="${pi/2} 0 0"/>
         <geometry><cylinder radius="${wheel_radius}" length="${wheel_width}"/></geometry>
         <material name="black"/>
       </visual>
       <collision>
+        <origin xyz="0 0 0" rpy="${pi/2} 0 0"/>
         <geometry><cylinder radius="${wheel_radius}" length="${wheel_width}"/></geometry>
       </collision>
     </link>
-    <joint name="${prefix}_wheel_joint" type="continuous">
+    <joint name="${name}_wheel_joint" type="continuous">
       <parent link="base_link"/>
-      <child link="${prefix}_wheel_link"/>
-      <origin xyz="${-wheelbase/2} ${y_offset} ${-base_height/2}" rpy="${-pi/2} 0 0"/>
-      <axis xyz="0 0 1"/>
+      <child link="${name}_wheel_link"/>
+      <origin xyz="${-base_length/3} ${y} ${wheel_radius + 0.005}"/>
+      <axis xyz="0 1 0"/>
     </joint>
+    <gazebo reference="${name}_wheel_link">
+      <!-- <mu1>1.0</mu1>
+      <mu2>1.0</mu2> -->
+      <!-- <kp>300000.0</kp>
+      <kd>50.0</kd> -->
+    </gazebo>
   </xacro:macro>
-  <xacro:rear_wheel prefix="rear_left"  y_offset="${track/2}"/>
-  <xacro:rear_wheel prefix="rear_right" y_offset="${-track/2}"/>
-  <xacro:macro name="front_wheel" params="prefix y_offset">
-    <link name="${prefix}_steer_link">
-      <inertial>
-        <mass value="0.1"/>
-        <inertia ixx="0.01" ixy="0" ixz="0" iyy="0.01" iyz="0" izz="0.01"/>
-      </inertial>
-    </link>
-    <joint name="${prefix}_steer_joint" type="revolute">
-      <parent link="base_link"/>
-      <child link="${prefix}_steer_link"/>
-      <origin xyz="${wheelbase/2} ${y_offset} ${-base_height/2}" rpy="0 0 0"/>
-      <axis xyz="0 0 1"/>
-      <limit lower="-0.6" upper="0.6" effort="1000" velocity="100"/>
-    </joint>
-    <link name="${prefix}_wheel_link">
-      <xacro:cylinder_inertia m="${wheel_mass}" r="${wheel_radius}" h="${wheel_width}"/>
-      <visual>
-        <geometry><cylinder radius="${wheel_radius}" length="${wheel_width}"/></geometry>
-        <material name="black"/>
-      </visual>
-      <collision>
-        <geometry><cylinder radius="${wheel_radius}" length="${wheel_width}"/></geometry>
-      </collision>
-    </link>
-    <joint name="${prefix}_wheel_joint" type="continuous">
-      <parent link="${prefix}_steer_link"/>
-      <child link="${prefix}_wheel_link"/>
-      <origin xyz="0 0 0" rpy="${-pi/2} 0 0"/>
-      <axis xyz="0 0 1"/>
-    </joint>
-  </xacro:macro>
-  <xacro:front_wheel prefix="front_left"  y_offset="${track/2}"/>
-  <xacro:front_wheel prefix="front_right" y_offset="${-track/2}"/>
+  <xacro:wheel name="left"  y="${track/2}"/>
+  <xacro:wheel name="right" y="${-track/2}"/>
   <link name="camera_link">
     <visual>
@@ -105,9 +93,10 @@
       <material name="green"/>
     </visual>
+    <xacro:box_inertia m="0.1" x="${cam_size}" y="${cam_size}" z="${cam_size}"/>
   </link>
   <joint name="camera_joint" type="fixed">
-    <parent link="base_link"/>
+    <parent link="imu_link"/>
     <child link="camera_link"/>
-    <origin xyz="${base_length/2} 0 ${base_height/2 + cam_size/2}"/>
+    <origin xyz="0.375 0 0.125" rpy="0 0 0"/>
   </joint>
   <link name="camera_optical_frame"/>
@@ -117,42 +106,58 @@
     <origin xyz="0 0 0" rpy="${-pi/2} 0 ${-pi/2}"/>
   </joint>
+  <gazebo reference="camera_link">
+    <sensor name="/apriltag_slam/camera" type="camera">
+      <pose> 0 0 0 0 0 0 </pose>
+      <visualize>true</visualize>
+      <update_rate>10</update_rate>
+      <camera>
+        <horizontal_fov>1.089</horizontal_fov>
+        <image>
+          <format>R8G8B8</format>
+          <width>640</width>
+          <height>480</height>
+        </image>
+        <clip>
+          <near>0.05</near>
+          <far>8.0</far>
+        </clip>
+      </camera>
+      <plugin name="camera_controller" filename="libgazebo_ros_camera.so">
+        <frame_name>camera_optical_frame</frame_name>
+      </plugin>
+    </sensor>
+  </gazebo>
   <link name="imu_link"/>
   <joint name="imu_joint" type="fixed">
     <parent link="base_link"/>
     <child link="imu_link"/>
-    <origin xyz="0 0 0"/>
+    <origin xyz="0 0 ${base_height/2 + wheel_radius}"/>
   </joint>
-  <ros2_control name="AckermannSystem" type="system">
+  <gazebo reference="imu_link">
+    <sensor name="imu_sensor" type="imu">
+      <plugin name="imu_plugin" filename="libgazebo_ros_imu_sensor.so"/>
+      <always_on>true</always_on>
+      <update_rate>100</update_rate>
+      <imu/>
+    </sensor>
+  </gazebo>
+  <ros2_control name="DiffDriveSystem" type="system">
     <hardware>
       <plugin>gazebo_ros2_control/GazeboSystem</plugin>
     </hardware>
-    <joint name="front_left_steer_joint">
-      <command_interface name="position"/>
-      <state_interface name="position"/>
-      <state_interface name="velocity"/>
+    <joint name="left_wheel_joint">
+      <command_interface name="velocity"/>
+      <state_interface name="position"/><state_interface name="velocity"/>
     </joint>
-    <joint name="front_right_steer_joint">
-      <command_interface name="position"/>
-      <state_interface name="position"/>
-      <state_interface name="velocity"/>
+    <joint name="right_wheel_joint">
+      <command_interface name="velocity"/>
+      <state_interface name="position"/><state_interface name="velocity"/>
     </joint>
-    <joint name="rear_left_wheel_joint">
-      <command_interface name="velocity"/>
-      <state_interface name="velocity"/>
-      <state_interface name="position"/>
-    </joint>
-    <joint name="rear_right_wheel_joint">
-      <command_interface name="velocity"/>
-      <state_interface name="velocity"/>
-      <state_interface name="position"/>
-    </joint>
-    <joint name="front_left_wheel_joint">
-      <state_interface name="velocity"/>
-      <state_interface name="position"/>
-    </joint>
-    <joint name="front_right_wheel_joint">
-      <state_interface name="velocity"/>
-      <state_interface name="position"/>
-    </joint>
+    <sensor name="imu_sensor">
+        <state_interface name="orientation.x"/><state_interface name="orientation.y"/>
+        <state_interface name="orientation.z"/><state_interface name="orientation.w"/>
+        <state_interface name="angular_velocity.x"/><state_interface name="angular_velocity.y"/><state_interface name="angular_velocity.z"/>
+        <state_interface name="linear_acceleration.x"/><state_interface name="linear_acceleration.y"/><state_interface name="linear_acceleration.z"/>
+    </sensor>
   </ros2_control>
   <gazebo>
@@ -161,20 +166,3 @@
     </plugin>
   </gazebo>
-  <gazebo reference="camera_link">
-    <sensor name="camera" type="camera">
-      <always_on>true</always_on><update_rate>30.0</update_rate>
-      <camera><horizontal_fov>1.396</horizontal_fov><image><width>640</width><height>480</height><format>R8G8B8</format></image><clip><near>0.02</near><far>50.0</far></clip></camera>
-      <plugin name="camera_controller" filename="libgazebo_ros_camera.so">
-        <frame_name>camera_optical_frame</frame_name>
-      </plugin>
-    </sensor>
-  </gazebo>
-  <gazebo reference="imu_link">
-    <sensor name="imu_sensor" type="imu">
-      <plugin filename="libgazebo_ros_imu_sensor.so" name="imu_plugin">
-        <ros><namespace>/apriltag_slam/imu</namespace><remapping>~/out:=data_raw</remapping></ros>
-      </plugin>
-      <always_on>true</always_on><update_rate>100</update_rate>
-    </sensor>
-  </gazebo>
 </robot>

File: src/apriltag_slam/urdf/robot_effort.urdf.xacro (robot description, xacro)
@@ -36,5 +36,4 @@
     </inertial>
   </xacro:macro>
-  <!-- Base Footprint -->
   <link name="base_footprint"/>
   <joint name="base_joint" type="fixed">
@@ -196,7 +195,23 @@
     </plugin>
   </gazebo>
+  <gazebo>
+    <plugin name="gazebo_ros_p3d" filename="libgazebo_ros_p3d.so">
+      <ros>
+        <!-- Ensure the topic name matches your RViz settings -->
+        <remapping>odom:=/apriltag_slam/ground_truth/odom</remapping>
+      </ros>
+      <frame_name>world</frame_name>
+      <body_name>imu_link</body_name>
+      <update_rate>50.0</update_rate>
+      <gaussian_noise>0.01</gaussian_noise>
+      <xyz_offset>0 0 0</xyz_offset>
+      <rpy_offset>0 0 0</rpy_offset>
+      <!-- Sole broadcaster for world -> base_footprint -->
+      <publish_odom_tf>true</publish_odom_tf>
+    </plugin>
+  </gazebo>
   <!-- Camera Sensor -->
   <gazebo reference="camera_link">
-    <sensor name="camera" type="camera">
+    <sensor name="/apriltag_slam/camera" type="camera">
       <always_on>true</always_on>
       <update_rate>30.0</update_rate>
